Commit message: fix: modify urdf of  wheels and sensor

File: my_robot/urdf/my_robot.xacro (robot description, xacro)
@@ -29,4 +29,7 @@
         <box size=".4 .2 .1"/>
       </geometry>
+    <material name='blue'>
+    <color rgba="0 0 1.0 1.0" />
+    </material>
     </visual>
     <collision name='back_caster_collision'>
@@ -62,10 +65,12 @@
   </inertial>
   <collision>
-  <geometry >
+  <origin xyz="0 0 0" rpy="0.0 1.5707 1.5707"/>
+  <geometry>
   <cylinder  radius="0.1" length="0.05" />
   </geometry>
   </collision>
   <visual>
-  <geometry >
+  <origin xyz="0 0 0" rpy="0.0 1.5707 1.5707"/>
+  <geometry>
   <cylinder  radius="0.1" length="0.05" />
   </geometry>
@@ -79,10 +84,12 @@
   </inertial>
   <collision>
-  <geometry >
+  <origin xyz="0 0 0" rpy="0.0 1.5707 1.5707"/>
+  <geometry>
   <cylinder  radius="0.1" length="0.05" />
   </geometry>
   </collision>
   <visual>
-  <geometry >
+  <origin xyz="0 0 0" rpy="0.0 1.5707 1.5707"/>
+  <geometry>
   <cylinder  radius="0.1" length="0.05" />
   </geometry>
@@ -96,4 +103,5 @@
 </inertial>
 <collision>
+<origin xyz="0 0 0" rpy="0 0 0"/>
 <geometry>
 <box size="0.05 0.05 0.05"/>
@@ -101,4 +109,5 @@
 </collision>
 <visual>
+<origin xyz="0 0 0" rpy="0 0 0"/>
 <geometry>
 <box size="0.05 0.05 0.05"/>
@@ -113,4 +122,5 @@
 </inertial>
 <collision>
+<origin xyz="0 0 0" rpy="0 0 0"/>
 <geometry>
 <box size="0.1 0.1 0.1"/>
@@ -118,5 +128,8 @@
 </collision>
 <visual>
-<geometry filename ="package://my_robot/meshes/hokuyo.dae"/>
+<origin xyz="0 0 0" rpy="0 0 0"/>
+<geometry>
+<mesh filename ="package://my_robot/meshes/hokuyo.dae" scale="1 1 1"/>
+</geometry>
 </visual>
 </link>
@@ -125,5 +138,5 @@
 <parent link="chassis"/>
 <child link="hokuyo"/>
-<axis xyz="0 1 0" rpy="0 0 0"/>
+<axis xyz="0 1 0"/>
 </joint>
 <joint type="fixed" name="camera_joint">
@@ -131,5 +144,5 @@
 <parent link="chassis"/>
 <child link="camera" />
-<axis xyz="0 1 0" rpy="0 0 0"/>
+<axis xyz="0 1 0" />
 </joint>
 <joint type="continuous" name="right_wheel_hinge">
@@ -137,5 +150,5 @@
 <child link="right_wheel" />
 <parent link="chassis" />
-<axis xyz="0 1 0" rpy="0 0 0"/>
+<axis xyz="0 1 0" />
 <limit effort="10000" velocity="1000" />
 <dynamics damping="1.0" friction="1.0" />
@@ -145,5 +158,5 @@
 <child link="left_wheel" />
 <parent link="chassis" />
-<axis xyz="0 1 0" rpy="0 0 0"/>
+<axis xyz="0 1 0"/>
 <limit effort="10000" velocity="1000" />
 <dynamics damping="1.0" friction="1.0" />
